File: HW/PCB/micShield.sch (EAGLE design)
At the start: 43 parts, among them M1 PMM-3738-VM1010-R, U1 LM27762DSSR, U2 LT6002CGN

Commit message: More updates to schematics and layout.
Parts:
- added R12: (no value), SparkFun-Resistors:RESISTOR0402
Connections:
- net DOUT: now also U$1.34/A15
- net GA1: now also R12.1
- net GA2: now also R12.2
- net MODE: now also U$1.33/A14
Changed lines of the file:
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@@
 <part name="R9" library="SparkFun-Resistors" deviceset="RESISTOR" device="0402"/>
 <part name="R10" library="SparkFun-Resistors" deviceset="RESISTOR" device="0402"/>
+<part name="R12" library="SparkFun-Resistors" deviceset="RESISTOR" device="0402"/>
 </parts>
 <sheets>
@@
 <instance part="R9" gate="G$1" x="335.28" y="78.74" rot="R90"/>
 <instance part="R10" gate="G$1" x="327.66" y="73.66" rot="R180"/>
+<instance part="R12" gate="G$1" x="228.6" y="60.96" rot="R180"/>
 </instances>
 <busses>
@@
 <label x="215.9" y="35.56" size="1.778" layer="95" rot="MR0"/>
 </segment>
+<segment>
+<pinref part="U$1" gate="G$1" pin="33/A14"/>
+<wire x1="314.96" y1="15.24" x2="317.5" y2="15.24" width="0.1524" layer="91"/>
+<label x="317.5" y="15.24" size="1.778" layer="95"/>
+</segment>
 </net>
 <net name="GA1" class="0">
@@
 <label x="215.9" y="38.1" size="1.778" layer="95" rot="MR0"/>
 </segment>
+<segment>
+<pinref part="R12" gate="G$1" pin="1"/>
+<wire x1="233.68" y1="60.96" x2="241.3" y2="60.96" width="0.1524" layer="91"/>
+<label x="241.3" y="60.96" size="1.778" layer="95"/>
+</segment>
 </net>
 <net name="GA2" class="0">
@@
 <wire x1="218.44" y1="40.64" x2="215.9" y2="40.64" width="0.1524" layer="91"/>
 <label x="215.9" y="40.64" size="1.778" layer="95" rot="MR0"/>
+</segment>
+<segment>
+<pinref part="R12" gate="G$1" pin="2"/>
+<wire x1="223.52" y1="60.96" x2="215.9" y2="60.96" width="0.1524" layer="91"/>
+<label x="215.9" y="60.96" size="1.778" layer="95" rot="MR0"/>
 </segment>
 </net>
@@
 <label x="241.3" y="43.18" size="1.778" layer="95"/>
 </segment>
-</net>
+<segment>
+<pinref part="U$1" gate="G$1" pin="34/A15"/>
+<wire x1="314.96" y1="17.78" x2="317.5" y2="17.78" width="0.1524" layer="91"/>
+<label x="317.5" y="17.78" size="1.778" layer="95"/>
+</segment>
+</net>

Commit message: Woohoo. Version 0.1 ordered.
Parts:
- added FRAME1, FRAME2: FRAME-LETTER, SparkFun-Aesthetics:FRAME-LETTER
- added TP1, TP2, TP3, TP4, TP5, TP6: TEST-POINT3, SparkFun-Passives:TEST-POINT3
Connections:
- net DOUT: now also TP6.1
- net GA1: now also TP3.1
- net GA2: now also TP2.1
- net MODE: now also TP4.1
- net TO_AMP: now also TP5.1
- net V3_3P: now also TP1.1
Other:
- moved on the sheet: C4, C6, C7, M1, R1, R11, R12, R14, R15, R16, R17, R18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
